Commit message: fix

File: src/andino/andino_description/urdf/include/andino_control.urdf.xacro (robot description, xacro)
@@ -33,5 +33,5 @@
         <state_interface name="position"/>
       </joint>
-      <joint name="ultrasonic_sensor">
+      <joint name="ultrasonic_joint">
         <state_interface name="range"/>
       </joint>
