Commit message: Sync updated files from Raspberry Pi to repository

File: src/andino/andino_description/urdf/andino.urdf.xacro (robot description, xacro)
@@ -1,20 +1,14 @@
 <?xml version="1.0"?>
 <robot xmlns:xacro="http://www.ros.org/wiki/xacro" name="andino">
-  <!-- ====== General Properties ====== -->
   <xacro:property name="package_name" value="andino_description"/>
   <xacro:property name="robot_name" value="andino"/>
-  <!-- ====== Include Macros ====== -->
   <xacro:include filename="$(find ${package_name})/urdf/include/common_macros.urdf.xacro" />
   <xacro:include filename="$(find ${package_name})/urdf/include/common_sensors.urdf.xacro" />
   <xacro:include filename="$(find ${package_name})/urdf/include/andino_caster_macro.urdf.xacro" />
-  <!-- ====== Arguments ====== -->
   <xacro:arg name="yaml_config_dir" default="$(find ${package_name})/config/${robot_name}" />
+  <xacro:property name="caster_wheel_yaml" value="$(arg yaml_config_dir)/caster_wheel.yaml" />
+  <xacro:property name="caster_wheel_props" value="${xacro.load_yaml(caster_wheel_yaml)}"/>
   <xacro:arg name="use_fixed_caster" default="True"/>
   <xacro:arg name="use_real_ros_control" default="True"/>
-  <!-- Enable/disable ultrasonic sensor (default ON so it works without passing args from launch) -->
-  <xacro:arg name="use_ultrasonic" default="True"/>
-  <!-- ====== Load YAML Configs ====== -->
-  <xacro:property name="caster_wheel_yaml" value="$(arg yaml_config_dir)/caster_wheel.yaml" />
-  <xacro:property name="caster_wheel_props" value="${xacro.load_yaml(caster_wheel_yaml)}"/>
   <xacro:property name="wheel_yaml" value="$(arg yaml_config_dir)/wheel.yaml" />
   <xacro:property name="wheel_props" value="${xacro.load_yaml(wheel_yaml)}"/>
@@ -29,40 +23,56 @@
   <xacro:property name="hardware_yaml" value="$(arg yaml_config_dir)/hardware.yaml" />
   <xacro:property name="hardware_props" value="${xacro.load_yaml(hardware_yaml)}"/>
-  <!-- ====== Footprint ====== -->
+  <!-- Footprint link -->
   <xacro:footprint wheel_props="${wheel_props}" />
-  <!-- ====== Base link ====== -->
-  <xacro:base link_name="base_link" base_prop="${base_props}" mesh="${base_props['base']['mesh']}">
+  <!-- Base link -->
+  <xacro:base link_name="base_link" base_prop="${base_props}" mesh="${base_props['base']['mesh']}" >
     <origin xyz="0 0 0" rpy="0 0 0" />
   </xacro:base>
-  <!-- ====== Second base link ====== -->
-  <xacro:base link_name="second_base_link" base_prop="${second_base_props}" mesh="${second_base_props['base']['mesh']}">
-    <origin xyz="0 0 0.05" rpy="0 0 0" />
+  <!-- Second story link -->
+  <xacro:base link_name="second_base_link" base_prop="${second_base_props}" mesh="${second_base_props['base']['mesh']}" >
+    <origin xyz="0 0 0.254" rpy="0 0 0" />
   </xacro:base>
-  <!-- Fixed joint connecting second base to base link -->
+  <!-- Joint to connect second_story with base_link -->
   <joint name="second_base_joint" type="fixed">
     <parent link="base_link"/>
-    <child link="second_base_link"/>
-    <origin xyz="0 0 0" rpy="0 0 0"/>
+    <child link="second_base_link" />
+    <origin xyz="0 0 0" rpy="0 0 0" />
   </joint>
-  <!-- ====== Caster Wheel ====== -->
-  <xacro:caster_wheel
-      reflect="-1"
-      use_fixed="$(arg use_fixed_caster)"
-      wheel_props="${caster_wheel_props}" />
-  <!-- ====== Wheels ====== -->
-  <xacro:wheel prefix="right" reflect="-1" wheel_props="${wheel_props}" base_props="${base_props}" />
-  <xacro:wheel prefix="left"  reflect="1"  wheel_props="${wheel_props}" base_props="${base_props}" />
-  <!-- ====== Motors ====== -->
-  <xacro:motor prefix="right" reflect="-1" motor_props="${motor_props}" base_props="${base_props}" />
-  <xacro:motor prefix="left"  reflect="1"  motor_props="${motor_props}" base_props="${base_props}" />
-  <!-- ====== Sensors ====== -->
-  <xacro:laser prefix="rplidar" parent_link="second_base_link" sensor_prop="${sensor_prop}" />
-  <xacro:camera_sensor parent_link="base_link" sensor_prop="${sensor_prop}" />
-  <xacro:imu_sensor    parent_link="base_link" sensor_prop="${sensor_prop}" />
-  <!-- Ultrasonic only if enabled -->
-  <xacro:if value="$(arg use_ultrasonic)">
-    <xacro:ultrasonic_sensor parent_link="base_link" sensor_prop="${sensor_prop}" />
-  </xacro:if>
-  <!-- ====== ROS 2 Control (hardware interfaces) ====== -->
+  <!-- Caster Wheel -->
+  <!-- Wheels -->
+  <xacro:wheel prefix="right" reflect="-1"
+                      wheel_props="${wheel_props}"
+                      base_props="${base_props}" >
+  </xacro:wheel>
+  <xacro:wheel prefix="left" reflect="1"
+                      wheel_props="${wheel_props}"
+                      base_props="${base_props}" >
+  </xacro:wheel>
+  <xacro:back_wheel prefix="right" reflect="-1"
+                      wheel_props="${wheel_props}"
+                      base_props="${base_props}" >
+  </xacro:back_wheel>
+  <xacro:back_wheel prefix="left" reflect="1"
+                      wheel_props="${wheel_props}"
+                      base_props="${base_props}" >
+  </xacro:back_wheel>
+  <!-- Motors -->
+  <xacro:motor prefix="right" reflect="-1"
+                      motor_props="${motor_props}"
+                      base_props="${base_props}" >
+  </xacro:motor>
+  <xacro:motor prefix="left" reflect="1"
+                      motor_props="${motor_props}"
+                      base_props="${base_props}" >
+  </xacro:motor>
+  <!-- Sensors -->
+  <xacro:laser prefix="rplidar" parent_link="base_link"
+                   sensor_prop="${sensor_prop}">
+  </xacro:laser>
+  <xacro:camera_sensor parent_link="base_link" sensor_prop="${sensor_prop}">
+  </xacro:camera_sensor>
+<xacro:imu_sensor parent_link="base_link" sensor_prop="${sensor_prop}">
+  </xacro:imu_sensor>
+  <!-- ros2_control -->
   <xacro:if value="$(arg use_real_ros_control)">
     <xacro:include filename="$(find ${package_name})/urdf/include/andino_control.urdf.xacro" />

File: src/andino/andino_description/urdf/include/andino_control.urdf.xacro (robot description, xacro)
@@ -16,9 +16,10 @@
         <param name="timeout">${hardware_props['timeout']}</param>
         <param name="enc_ticks_per_rev">${hardware_props['enc_ticks_per_rev']}</param>
+        <param name="imu_sensor_name">imu_sensor</param>
       </hardware>
       <joint name="left_wheel_joint">
         <command_interface name="velocity">
-          <param name="min">-5</param>
-          <param name="max">5</param>
+          <param name="min">-10</param>
+          <param name="max">10</param>
         </command_interface>
         <state_interface name="velocity"/>
@@ -27,10 +28,19 @@
       <joint name="right_wheel_joint">
         <command_interface name="velocity">
-          <param name="min">-5</param>
-          <param name="max">5</param>
+          <param name="min">-10</param>
+          <param name="max">10</param>
         </command_interface>
         <state_interface name="velocity"/>
         <state_interface name="position"/>
       </joint>
+      <sensor name="imu_sensor">
+      <state_interface name="angular_velocity.x"/>
+      <state_interface name="angular_velocity.y"/>
+      <state_interface name="angular_velocity.z"/>
+      <state_interface name="linear_acceleration.x"/>
+      <state_interface name="linear_acceleration.y"/>
+      <state_interface name="linear_acceleration.z"/>
+      <param name="frame_id">imu_link</param>
+      </sensor>
     </ros2_control>
   </xacro:macro>

File: src/andino/andino_description/urdf/include/common_macros.urdf.xacro (robot description, xacro)
@@ -13,5 +13,5 @@
                params="prefix reflect wheel_props base_props ">
   <xacro:property name="pos_x_joint"
-     value="${(base_props['base']['x_size']/2) - wheel_props['x_offset']}"/>
+     value="${(wheel_props['x_offset'])}"/>
   <xacro:property name="pos_y_joint"
     value="${(base_props['base']['y_size']/2) + wheel_props['y_offset'] + (wheel_props['length']/2)}"/>
@@ -62,4 +62,56 @@
     </joint>
   </xacro:macro>
+  <xacro:macro name="back_wheel"
+               params="prefix reflect wheel_props base_props ">
+  <xacro:property name="pos_x_joint"
+     value="${(wheel_props['x_offset'])}"/>
+  <xacro:property name="pos_y_joint"
+    value="${(base_props['base']['y_size']/2) + wheel_props['y_offset'] + (wheel_props['length']/2)}"/>
+  <xacro:property name="pos_z_joint" value="${wheel_props['z_offset']}"/>
+    <link name="${prefix}_back_wheel">
+    <xacro:if value="${wheel_props['mesh'] != '' }" >
+      <visual>
+        <origin xyz="0.0 0 0" rpy="${pi/2} 0 ${pi/2.0*(reflect - 1)}"/>
+        <geometry>
+          <xacro:if value="${wheel_props['scale'] == '' }" >
+            <mesh filename="package://andino_description/meshes/${robot_name}/${wheel_props['mesh']}" />
+          </xacro:if>
+          <xacro:unless value="${wheel_props['scale'] == '' }" >
+            <mesh filename="package://andino_description/meshes/${robot_name}/${wheel_props['mesh']}" scale="${wheel_props['scale']}" />
+          </xacro:unless>
+        </geometry>
+        <material name="dark_grey"/>
+      </visual>
+    </xacro:if>
+    <xacro:if value="${wheel_props['mesh'] == '' }" >
+      <visual>
+        <origin xyz="0.0 0 0" rpy="${pi/2} 0 0"/>
+         <geometry>
+         <cylinder radius="${wheel_props['radius']}" length="${wheel_props['length']}"/>
+        </geometry>
+        <material name="red"/>
+      </visual>
+    </xacro:if>
+      <collision>
+        <origin xyz="0 0 0" rpy="${pi/2} 0 0"/>
+        <geometry>
+          <cylinder radius="${wheel_props['radius']}" length="${wheel_props['length']}"/>
+        </geometry>
+      </collision>
+      <xacro:cylinder_inertia m="${wheel_props['mass']}"
+                              r="${wheel_props['radius']}"
+                              l="${wheel_props['length']}"
+                              o_xyz="0.0 0.0 0.0"
+                              o_rpy="${pi/2.0} 0.0 0.0" >
+      </xacro:cylinder_inertia>
+    </link>
+    <joint name="${prefix}_back_wheel_joint" type="continuous">
+      <axis xyz="0 1 0" rpy="0 0 0" />
+      <parent link="base_link"/>
+      <child link="${prefix}_back_wheel"/>
+      <origin xyz="${pos_x_joint-0.29} ${reflect* pos_y_joint} ${pos_z_joint}" rpy="0 0 0"/>
+      <mimic joint="${prefix}_wheel_joint" multiplier="1"/>
+    </joint>
+  </xacro:macro>
 <!-- ===================== Motor xacro =========================================
   params:
@@ -76,5 +128,5 @@
      value="${(base_props['base']['x_size']/2) - motor_props['x_offset']}"/>
   <xacro:property name="pos_y_joint"
-    value="${(base_props['base']['y_size']/2) + motor_props['y_offset'] + (motor_props['y_size']/2)}"/>
+    value="${(base_props['base']['y_size']/2) + motor_props['y_offset'] + (motor_props['length']/2)}"/>
   <xacro:property name="pos_z_joint" value="${motor_props['z_offset']}"/>
     <link name="${prefix}_motor">
@@ -97,5 +149,5 @@
         <origin xyz="0.0 0 0" rpy="${pi/2} 0 0"/>
          <geometry>
-          <box size="${motor_props['x_size']} ${motor_props['y_size']} ${motor_props['z_size']}"/>
+          <cylinder radius="${motor_props['radius']}" length="${motor_props['length']}"/>
         </geometry>
         <material name="red"/>
@@ -105,17 +157,16 @@
         <origin xyz="0 0 0" rpy="${pi/2} 0 0"/>
         <geometry>
-          <box size="${motor_props['x_size']} ${motor_props['y_size']} ${motor_props['z_size']}"/>
+          <cylinder radius="${motor_props['radius']}" length="${motor_props['length']}"/>
         </geometry>
       </collision>
-      <xacro:box_inertia m="${motor_props['mass']}"
-                         x="${motor_props['x_size']}"
-                         y="${motor_props['y_size']}"
-                         z="${motor_props['z_size']}">
-      </xacro:box_inertia>
+      <xacro:cylinder_inertia m="${motor_props['mass']}"
+                         r="${motor_props['radius']}"
+                         l="${motor_props['length']}">
+      </xacro:cylinder_inertia>
     </link>
     <joint name="${prefix}_motor_joint" type="fixed">
       <parent link="base_link"/>
       <child link="${prefix}_motor"/>
-      <origin xyz="${pos_x_joint} ${reflect* pos_y_joint} ${pos_z_joint}" rpy="0 ${-pi/2.0*(reflect - 1)} 0"/>
+      <origin xyz="${pos_x_joint} ${reflect* pos_y_joint} ${pos_z_joint}" rpy="0 0 0"/>
       <axis xyz="0 1 0" rpy="0 0 0" />
     </joint>
@@ -183,7 +234,7 @@
     <!-- Joint to connect base_footprint with base_link -->
     <joint name="base_footprint_joint" type="fixed">
-      <parent link="base_link"/>
-      <child link="base_footprint" />
-      <origin xyz="0 0 ${-(wheel_props['radius'] - wheel_props['z_offset'])}" rpy="0 0 0" />
+      <parent link="base_footprint"/>
+      <child link="base_link" />
+      <origin xyz="0 0 ${(wheel_props['radius'] - wheel_props['z_offset'])}" rpy="0 0 0" />
     </joint>
   </xacro:macro>
