Commit message: back old

File: src/andino/andino_description/urdf/include/common_sensors.urdf.xacro (robot description, xacro)
@@ -1,114 +1,181 @@
 <?xml version="1.0"?>
 <robot xmlns:xacro="http://www.ros.org/wiki/xacro">
-<xacro:macro name="laser" params="prefix parent_link sensor_prop">
-  <xacro:property name="mesh"
-     value="${sensor_prop['laser']['mesh']}"/>
-  <link name="${prefix}_laser_link">
-    <xacro:if value="${mesh != '' }" >
-    <visual>
-      <origin xyz="0 0 0" rpy="0 0 ${pi}"/>
-      <geometry>
-        <mesh filename="package://andino_description/meshes/sensors/${mesh}" />
-      </geometry>
-      <material name="dark_grey"/>
-    </visual>
-  </xacro:if>
-  <xacro:if value="${mesh == '' }" >
-    <visual>
-      <origin xyz="0 0 0" rpy="0 0 0"/>
-        <geometry>
-        <cylinder radius="${sensor_prop['laser']['radius']}" length="${sensor_prop['laser']['length']}"/>
-      </geometry>
-      <material name="red"/>
-    </visual>
-  </xacro:if>
-    <collision>
-      <origin xyz="0 0 0" rpy="0 0 0"/>
-      <geometry>
-        <cylinder radius="${sensor_prop['laser']['radius']}" length="${sensor_prop['laser']['length']}"/>
-      </geometry>
-    </collision>
-    <xacro:cylinder_inertia m="${sensor_prop['laser']['mass']}"
-                            r="${sensor_prop['laser']['radius']}"
-                            l="${sensor_prop['laser']['length']}"
-                            o_xyz="0 0 0"
-                            o_rpy="0 0 0" />
-  </link>
-  <joint name="${prefix}_laser_joint" type="fixed">
-    <parent link="${parent_link}"/>
-    <child link="${prefix}_laser_link"/>
-    <origin xyz="${sensor_prop['laser']['dx']} ${sensor_prop['laser']['dy']} ${sensor_prop['laser']['dz']}" rpy="0 0 ${pi}"/>
-    <axis xyz="0 1 0" />
-  </joint>
-</xacro:macro>
-<xacro:macro name="camera_sensor" params="parent_link sensor_prop">
-  <xacro:property name="mesh"
-     value="${sensor_prop['camera']['mesh']}"/>
-  <link name="camera_link">
-    <xacro:if value="${mesh != '' }" >
-      <visual>
+  <!-- ===== Laser Macro ===== -->
+  <xacro:macro name="laser" params="prefix parent_link sensor_prop">
+    <xacro:property name="mesh" value="${sensor_prop['laser']['mesh']}"/>
+    <link name="${prefix}_laser_link">
+      <xacro:if value="${mesh != '' }">
+        <visual>
+          <origin xyz="0 0 0" rpy="0 0 ${pi}"/>
+          <geometry>
+            <mesh filename="package://andino_description/meshes/sensors/${mesh}" />
+          </geometry>
+          <material name="dark_grey"/>
+        </visual>
+      </xacro:if>
+      <xacro:if value="${mesh == '' }">
+        <visual>
+          <origin xyz="0 0 0" rpy="0 0 0"/>
+          <geometry>
+            <cylinder radius="${sensor_prop['laser']['radius']}" length="${sensor_prop['laser']['length']}"/>
+          </geometry>
+          <material name="red"/>
+        </visual>
+      </xacro:if>
+      <collision>
         <origin xyz="0 0 0" rpy="0 0 0"/>
         <geometry>
-          <mesh filename="package://andino_description/meshes/sensors/${mesh}" />
+          <cylinder radius="${sensor_prop['laser']['radius']}" length="${sensor_prop['laser']['length']}"/>
         </geometry>
-        <material name="blue"/>
-      </visual>
-    </xacro:if>
-    <xacro:if value="${mesh == '' }" >
-      <visual>
+      </collision>
+      <xacro:cylinder_inertia
+        m="${sensor_prop['laser']['mass']}"
+        r="${sensor_prop['laser']['radius']}"
+        l="${sensor_prop['laser']['length']}"
+        o_xyz="0 0 0"
+        o_rpy="0 0 0" />
+    </link>
+    <joint name="${prefix}_laser_joint" type="fixed">
+      <parent link="${parent_link}"/>
+      <child link="${prefix}_laser_link"/>
+      <origin xyz="${sensor_prop['laser']['dx']} ${sensor_prop['laser']['dy']} ${sensor_prop['laser']['dz']}" rpy="0 0 ${pi}"/>
+      <axis xyz="0 1 0" />
+    </joint>
+  </xacro:macro>
+  <!-- ===== Camera Macro (classic plugin kept as-is) ===== -->
+  <xacro:macro name="camera_sensor" params="parent_link sensor_prop">
+    <xacro:property name="mesh" value="${sensor_prop['camera']['mesh']}"/>
+    <link name="camera_link">
+      <!-- Visual -->
+      <xacro:if value="${mesh != '' }">
+        <visual>
+          <origin xyz="0 0 0" rpy="0 0 0"/>
+          <geometry>
+            <mesh filename="package://andino_description/meshes/sensors/${mesh}" />
+          </geometry>
+          <material name="blue"/>
+        </visual>
+      </xacro:if>
+      <xacro:if value="${mesh == '' }">
+        <visual>
+          <origin xyz="0 0 0" rpy="0 0 0"/>
+          <geometry>
+            <box size="${sensor_prop['camera']['box_size']} ${sensor_prop['camera']['box_size']} ${sensor_prop['camera']['box_size']}"/>
+          </geometry>
+          <material name="blue"/>
+        </visual>
+      </xacro:if>
+      <!-- Collision -->
+      <collision>
         <origin xyz="0 0 0" rpy="0 0 0"/>
         <geometry>
           <box size="${sensor_prop['camera']['box_size']} ${sensor_prop['camera']['box_size']} ${sensor_prop['camera']['box_size']}"/>
         </geometry>
-        <material name="blue"/>
+      </collision>
+      <!-- Inertia -->
+      <xacro:box_inertia
+        m="${sensor_prop['camera']['mass']}"
+        x="${sensor_prop['camera']['box_size']}"
+        y="${sensor_prop['camera']['box_size']}"
+        z="${sensor_prop['camera']['box_size']}"
+        o_xyz="0 0 0"
+        o_rpy="0 0 0" />
+      <!-- Classic Gazebo camera plugin (compatibility) -->
+      <gazebo>
+        <plugin name="camera_controller" filename="libgazebo_ros_camera.so">
+          <robotNamespace>/camera_front</robotNamespace>
+          <cameraName>camera_front</cameraName>
+          <imageTopicName>image_raw</imageTopicName>
+          <frameName>camera_link</frameName>
+          <updateRate>30.0</updateRate>
+          <alwaysOn>true</alwaysOn>
+        </plugin>
+      </gazebo>
+    </link>
+    <joint name="camera_joint" type="fixed">
+      <parent link="${parent_link}"/>
+      <child link="camera_link"/>
+      <origin xyz="${sensor_prop['camera']['dx']} ${sensor_prop['camera']['dy']} ${sensor_prop['camera']['dz']}" rpy="0 0 0"/>
+      <axis xyz="0 1 0" />
+    </joint>
+  </xacro:macro>
+  <!-- ===== IMU Macro (native sensor) ===== -->
+  <xacro:macro name="imu_sensor" params="parent_link sensor_prop">
+    <link name="imu_link">
+      <visual>
+        <geometry>
+          <box size="0.01 0.01 0.0025"/>
+        </geometry>
       </visual>
-    </xacro:if>
+      <collision>
+        <geometry>
+          <box size="0.01 0.01 0.0025"/>
+        </geometry>
+      </collision>
+      <inertial>
+        <mass value="1e-5" />
+        <origin xyz="0 0 0" rpy="0 0 0"/>
+        <inertia ixx="1e-6" ixy="0" ixz="0" iyy="1e-6" iyz="0" izz="1e-6" />
+      </inertial>
+      <sensor name="imu_sensor" type="imu">
+        <always_on>true</always_on>
+        <update_rate>50</update_rate>
+        <topic>/imu/data</topic>
+        <imu/>
+      </sensor>
+    </link>
+    <joint name="imu_joint" type="fixed">
+      <parent link="${parent_link}"/>
+      <child link="imu_link"/>
+      <origin xyz="${sensor_prop['imu']['dx']} ${sensor_prop['imu']['dy']} ${sensor_prop['imu']['dz']}" rpy="0 0 0"/>
+      <axis xyz="0 1 0" />
+    </joint>
+  </xacro:macro>
+  <!-- ===== Ultrasonic Macro (native single-beam ray) ===== -->
+<xacro:macro name="ultrasonic_sensor" params="parent_link sensor_prop">
+  <!-- Visual/Collision/Inertial link -->
+  <link name="ultrasonic_link">
+    <visual>
+      <geometry>
+        <box size="${sensor_prop['ultrasonic']['box_size']} ${sensor_prop['ultrasonic']['box_size']} ${sensor_prop['ultrasonic']['box_size']}"/>
+      </geometry>
+    </visual>
     <collision>
-      <origin xyz="0 0 0" rpy="0 0 0"/>
       <geometry>
-        <box size="${sensor_prop['camera']['box_size']} ${sensor_prop['camera']['box_size']} ${sensor_prop['camera']['box_size']}"/>
+        <box size="${sensor_prop['ultrasonic']['box_size']} ${sensor_prop['ultrasonic']['box_size']} ${sensor_prop['ultrasonic']['box_size']}"/>
       </geometry>
     </collision>
-    <xacro:box_inertia m="${sensor_prop['camera']['mass']}"
-                            x="${sensor_prop['camera']['box_size']}"
-                            y="${sensor_prop['camera']['box_size']}"
-                            z="${sensor_prop['camera']['box_size']}"
-                            o_xyz="0 0 0"
-                            o_rpy="0 0 0" />
+    <inertial>
+      <mass value="${sensor_prop['ultrasonic']['mass']}"/>
+      <origin xyz="0 0 0" rpy="0 0 0"/>
+      <inertia ixx="1e-6" ixy="0" ixz="0" iyy="1e-6" iyz="0" izz="1e-6"/>
+    </inertial>
+    <!-- SENSOR MUST BE A DIRECT CHILD OF <link> IN GZ -->
+    <sensor name="ultrasonic_front" type="ray">
+      <always_on>true</always_on>
+      <update_rate>20</update_rate>
+      <visualize>true</visualize>
+      <!-- اترك الـ topic محذوف هنا عشان GZ يولّد المسار التلقائي -->
+      <ray>
+        <scan>
+          <horizontal>
+            <samples>3</samples>
+            <resolution>1</resolution>
+            <min_angle>-0.017</min_angle>  <!-- ~ -1 deg -->
+            <max_angle>0.017</max_angle>   <!-- ~ +1 deg -->
+          </horizontal>
+        </scan>
+        <range>
+          <min>${sensor_prop['ultrasonic']['min_range']}</min>
+          <max>${sensor_prop['ultrasonic']['range']}</max>
+          <resolution>0.01</resolution>
+        </range>
+      </ray>
+    </sensor>
   </link>
-  <joint name="camera_joint" type="fixed">
+  <joint name="ultrasonic_joint" type="fixed">
     <parent link="${parent_link}"/>
-    <child link="camera_link"/>
-    <origin xyz="${sensor_prop['camera']['dx']} ${sensor_prop['camera']['dy']} ${sensor_prop['camera']['dz']}" rpy="0 0 0"/>
-    <axis xyz="0 1 0" />
-  </joint>
-</xacro:macro>
-<xacro:macro name="imu_sensor" params="parent_link sensor_prop">
-  <link name="imu_link">
-    <visual>
-      <origin xyz="0 0 0" rpy="0 0 0"/>
-      <geometry>
-        <box size="${sensor_prop['imu']['box_size_height']} ${sensor_prop['imu']['box_size']} 0.005"/>
-      </geometry>
-      <material name="black"/>
-    </visual>
-    <collision>
-      <origin xyz="0 0 0" rpy="0 0 0"/>
-      <geometry>
-        <box size="${sensor_prop['imu']['box_size']} ${sensor_prop['imu']['box_size']} ${sensor_prop['imu']['box_size_height']}"/>
-      </geometry>
-    </collision>
-    <xacro:box_inertia m="${sensor_prop['imu']['mass']}"
-                            x="${sensor_prop['imu']['box_size']}"
-                            y="${sensor_prop['imu']['box_size']}"
-                            z="${sensor_prop['imu']['box_size_height']}"
-                            o_xyz="0 0 0"
-                            o_rpy="0 0 0" />
-  </link>
-  <joint name="imu_joint" type="fixed">
-    <parent link="${parent_link}"/>
-    <child link="imu_link"/>
-    <origin xyz="${sensor_prop['imu']['dx']} ${sensor_prop['imu']['dy']} ${sensor_prop['imu']['dz']}" rpy="0 0 0"/>
-    <axis xyz="0 1 0" />
+    <child link="ultrasonic_link"/>
+    <origin xyz="${sensor_prop['ultrasonic']['dx']} ${sensor_prop['ultrasonic']['dy']} ${sensor_prop['ultrasonic']['dz']}" rpy="0 0 0"/>
   </joint>
 </xacro:macro>
