Commit message: final: everything wired up and working

File: src/andino/andino_description/urdf/andino.urdf.xacro (robot description, xacro)
@@ -1,20 +1,15 @@
 <?xml version="1.0"?>
-<robot xmlns:xacro="http://www.ros.org/wiki/xacro" name="andino">
-  <!-- ====== General Properties ====== -->
+<robot
+  name="Delivery Robot_urdf" xmlns:xacro="http://www.ros.org/wiki/xacro">
   <xacro:property name="package_name" value="andino_description"/>
   <xacro:property name="robot_name" value="andino"/>
-  <!-- ====== Include Macros ====== -->
   <xacro:include filename="$(find ${package_name})/urdf/include/common_macros.urdf.xacro" />
   <xacro:include filename="$(find ${package_name})/urdf/include/common_sensors.urdf.xacro" />
   <xacro:include filename="$(find ${package_name})/urdf/include/andino_caster_macro.urdf.xacro" />
-  <!-- ====== Arguments ====== -->
   <xacro:arg name="yaml_config_dir" default="$(find ${package_name})/config/${robot_name}" />
+  <xacro:property name="caster_wheel_yaml" value="$(arg yaml_config_dir)/caster_wheel.yaml" />
+  <xacro:property name="caster_wheel_props" value="${xacro.load_yaml(caster_wheel_yaml)}"/>
   <xacro:arg name="use_fixed_caster" default="True"/>
   <xacro:arg name="use_real_ros_control" default="True"/>
-  <!-- Enable/disable ultrasonic sensor (default ON so it works without passing args from launch) -->
-  <xacro:arg name="use_ultrasonic" default="True"/>
-  <!-- ====== Load YAML Configs ====== -->
-  <xacro:property name="caster_wheel_yaml" value="$(arg yaml_config_dir)/caster_wheel.yaml" />
-  <xacro:property name="caster_wheel_props" value="${xacro.load_yaml(caster_wheel_yaml)}"/>
   <xacro:property name="wheel_yaml" value="$(arg yaml_config_dir)/wheel.yaml" />
   <xacro:property name="wheel_props" value="${xacro.load_yaml(wheel_yaml)}"/>
@@ -29,40 +24,593 @@
   <xacro:property name="hardware_yaml" value="$(arg yaml_config_dir)/hardware.yaml" />
   <xacro:property name="hardware_props" value="${xacro.load_yaml(hardware_yaml)}"/>
-  <!-- ====== Footprint ====== -->
-  <xacro:footprint wheel_props="${wheel_props}" />
-  <!-- ====== Base link ====== -->
-  <xacro:base link_name="base_link" base_prop="${base_props}" mesh="${base_props['base']['mesh']}">
-    <origin xyz="0 0 0" rpy="0 0 0" />
-  </xacro:base>
-  <!-- ====== Second base link ====== -->
-  <xacro:base link_name="second_base_link" base_prop="${second_base_props}" mesh="${second_base_props['base']['mesh']}">
-    <origin xyz="0 0 0.05" rpy="0 0 0" />
-  </xacro:base>
-  <!-- Fixed joint connecting second base to base link -->
-  <joint name="second_base_joint" type="fixed">
-    <parent link="base_link"/>
-    <child link="second_base_link"/>
-    <origin xyz="0 0 0" rpy="0 0 0"/>
-  </joint>
-  <!-- ====== Caster Wheel ====== -->
-  <xacro:caster_wheel
-      reflect="-1"
-      use_fixed="$(arg use_fixed_caster)"
-      wheel_props="${caster_wheel_props}" />
-  <!-- ====== Wheels ====== -->
-  <xacro:wheel prefix="right" reflect="-1" wheel_props="${wheel_props}" base_props="${base_props}" />
-  <xacro:wheel prefix="left"  reflect="1"  wheel_props="${wheel_props}" base_props="${base_props}" />
-  <!-- ====== Motors ====== -->
-  <xacro:motor prefix="right" reflect="-1" motor_props="${motor_props}" base_props="${base_props}" />
-  <xacro:motor prefix="left"  reflect="1"  motor_props="${motor_props}" base_props="${base_props}" />
-  <!-- ====== Sensors ====== -->
-  <xacro:laser prefix="rplidar" parent_link="second_base_link" sensor_prop="${sensor_prop}" />
-  <xacro:camera_sensor parent_link="base_link" sensor_prop="${sensor_prop}" />
-  <xacro:imu_sensor    parent_link="base_link" sensor_prop="${sensor_prop}" />
-  <!-- Ultrasonic only if enabled -->
-  <xacro:if value="$(arg use_ultrasonic)">
-    <xacro:ultrasonic_sensor parent_link="base_link" sensor_prop="${sensor_prop}" />
-  </xacro:if>
-  <!-- ====== ROS 2 Control (hardware interfaces) ====== -->
+  <xacro:macro name="footprint"
+               params="wheel_props">
+    <!-- Base-Footprint -->
+    <!-- base_footprint is a fictitious link(frame) that is on the ground right below base_link origin -->
+    <link name="base_footprint" />
+    <!-- Joint to connect base_footprint with base_link -->
+    <joint name="base_footprint_joint" type="fixed">
+      <parent link="base_link"/>
+      <child link="base_footprint" />
+      <origin xyz="0 0 ${-(wheel_props['radius'] - wheel_props['z_offset'])}" rpy="0 0 0" />
+    </joint>
+  </xacro:macro>
+    <xacro:footprint wheel_props="${wheel_props}" />
+  <link
+    name="base_link">
+    <inertial>
+      <origin
+        xyz="0.0197110608215278 -0.0027804176800969 0.0969148643167121"
+        rpy="0 0 0" />
+      <mass
+        value="1.71386249919413" />
+      <inertia
+        ixx="0.0231569461000395"
+        ixy="2.50777808928108E-05"
+        ixz="0.000439253426777476"
+        iyy="0.038907074274843"
+        iyz="9.52977406661948E-06"
+        izz="0.0503099220851436" />
+    </inertial>
+    <visual>
+      <origin
+        xyz="0 0 0"
+        rpy="0 0 0" />
+      <geometry>
+        <mesh
+          filename="file:///home/mo/ws/src/andino/andino_description/meshes/base_link.STL" />
+      </geometry>
+      <material
+        name="">
+        <color
+          rgba="0 0 0 1" />
+      </material>
+    </visual>
+    <collision>
+      <origin
+        xyz="0 0 0"
+        rpy="0 0 0" />
+      <geometry>
+        <mesh
+          filename="file:///home/mo/ws/src/andino/andino_description/meshes/base_link.STL" />
+      </geometry>
+    </collision>
+  </link>
+  <link
+    name="left_wheel">
+    <inertial>
+      <origin
+        xyz="-1.43304923483356E-10 0.00578827480780619 2.09625126285085E-10"
+        rpy="0 0 0" />
+      <mass
+        value="0.468152044139992" />
+      <inertia
+        ixx="0.000602353929382081"
+        ixy="-7.18444193596074E-12"
+        ixz="-1.00167587643128E-11"
+        iyy="0.000954241002904411"
+        iyz="1.15813680205067E-12"
+        izz="0.000602353904161843" />
+    </inertial>
+    <visual>
+      <origin
+        xyz="0 0 0"
+        rpy="0 0 0" />
+      <geometry>
+        <mesh
+          filename="file:///home/mo/ws/src/andino/andino_description/meshes/left_wheel.STL" />
+      </geometry>
+      <material
+        name="">
+        <color
+          rgba="0.298039215686275 0.298039215686275 0.298039215686275 1" />
+      </material>
+    </visual>
+    <collision>
+      <origin
+        xyz="0 0 0"
+        rpy="0 0 0" />
+      <geometry>
+        <mesh
+          filename="file:///home/mo/ws/src/andino/andino_description/meshes/left_wheel.STL" />
+      </geometry>
+    </collision>
+  </link>
+  <joint
+    name="left_wheel_joint"
+    type="continuous">
+    <origin
+      xyz="0.14695 0.20151 -0.0138"
+      rpy="0 0 0" />
+    <parent
+      link="base_link" />
+    <child
+      link="left_wheel" />
+    <axis
+      xyz="0 1 0" />
+  </joint>
+  <link
+    name="right_wheel">
+    <inertial>
+      <origin
+        xyz="-1.16706644348596E-11 -0.00578827480780653 -2.53660450283411E-10"
+        rpy="0 0 0" />
+      <mass
+        value="0.468152044139995" />
+      <inertia
+        ixx="0.000602353913448942"
+        ixy="5.50210245429957E-12"
+        ixz="1.57577941586563E-11"
+        iyy="0.000954241002904415"
+        iyz="4.76280775920882E-12"
+        izz="0.000602353920094988" />
+    </inertial>
+    <visual>
+      <origin
+        xyz="0 0 0"
+        rpy="0 0 0" />
+      <geometry>
+        <mesh
+          filename="file:///home/mo/ws/src/andino/andino_description/meshes/right_wheel.STL" />
+      </geometry>
+      <material
+        name="">
+        <color
+          rgba="0.298039215686275 0.298039215686275 0.298039215686275 1" />
+      </material>
+    </visual>
+    <collision>
+      <origin
+        xyz="0 0 0"
+        rpy="0 0 0" />
+      <geometry>
+        <mesh
+          filename="file:///home/mo/ws/src/andino/andino_description/meshes/right_wheel.STL" />
+      </geometry>
+    </collision>
+  </link>
+  <joint
+    name="right_wheel_joint"
+    type="continuous">
+    <origin
+      xyz="0.14695 -0.20149 -0.0138"
+      rpy="0 0 0" />
+    <parent
+      link="base_link" />
+    <child
+      link="right_wheel" />
+    <axis
+      xyz="0 1 0" />
+  </joint>
+  <link
+    name="left_back_wheel">
+    <inertial>
+      <origin
+        xyz="5.29933874560129E-11 0.00578827480780614 -2.48335936883781E-10"
+        rpy="0 0 0" />
+      <mass
+        value="0.468152044139996" />
+      <inertia
+        ixx="0.00060235391871097"
+        ixy="6.20688903130094E-12"
+        ixz="-1.59872080469483E-11"
+        iyy="0.000954241002904416"
+        iyz="-3.79895060057837E-12"
+        izz="0.000602353914832962" />
+    </inertial>
+    <visual>
+      <origin
+        xyz="0 0 0"
+        rpy="0 0 0" />
+      <geometry>
+        <mesh
+          filename="file:///home/mo/ws/src/andino/andino_description/meshes/left_back_wheel.STL" />
+      </geometry>
+      <material
+        name="">
+        <color
+          rgba="0.298039215686275 0.298039215686275 0.298039215686275 1" />
+      </material>
+    </visual>
+    <collision>
+      <origin
+        xyz="0 0 0"
+        rpy="0 0 0" />
+      <geometry>
+        <mesh
+          filename="file:///home/mo/ws/src/andino/andino_description/meshes/left_back_wheel.STL" />
+      </geometry>
+    </collision>
+  </link>
+  <joint
+    name="left_back_wheel_joint"
+    type="continuous">
+    <origin
+      xyz="-0.14305 0.20001 -0.0138"
+      rpy="0 0 0" />
+    <parent
+      link="base_link" />
+    <child
+      link="left_back_wheel" />
+    <axis
+      xyz="0 1 0" />
+            <mimic joint="left_wheel_joint" multiplier="1"/>
+  </joint>
+  <link
+    name="right_back_wheel">
+    <inertial>
+      <origin
+        xyz="1.05106146008893E-10 -0.00578827480780619 -2.3115340544444E-10"
+        rpy="0 0 0" />
+      <mass
+        value="0.468152044139994" />
+      <inertia
+        ixx="0.000602353902050807"
+        ixy="2.73004690151346E-12"
+        ixz="6.52978696203657E-12"
+        iyy="0.000954241002904414"
+        iyz="6.74568812925498E-12"
+        izz="0.000602353931493122" />
+    </inertial>
+    <visual>
+      <origin
+        xyz="0 0 0"
+        rpy="0 0 0" />
+      <geometry>
+        <mesh
+          filename="file:///home/mo/ws/src/andino/andino_description/meshes/right_back_wheel.STL" />
+      </geometry>
+      <material
+        name="">
+        <color
+          rgba="0.298039215686275 0.298039215686275 0.298039215686275 1" />
+      </material>
+    </visual>
+    <collision>
+      <origin
+        xyz="0 0 0"
+        rpy="0 0 0" />
+      <geometry>
+        <mesh
+          filename="file:///home/mo/ws/src/andino/andino_description/meshes/right_back_wheel.STL" />
+      </geometry>
+    </collision>
+  </link>
+  <joint
+    name="right_back_wheel_joint"
+    type="continuous">
+    <origin
+      xyz="-0.14305 -0.20149 -0.0138"
+      rpy="0 0 0" />
+    <parent
+      link="base_link" />
+    <child
+      link="right_back_wheel" />
+    <axis
+      xyz="0 -1 0" />
+            <mimic joint="right_wheel_joint" multiplier="1"/>
+  </joint>
+  <link
+    name="front_left_motor_Link">
+    <inertial>
+      <origin
+        xyz="-2.93427859787698E-09 -0.0282987057433313 1.98829454782501E-07"
+        rpy="0 0 0" />
+      <mass
+        value="0.0243780634374845" />
+      <inertia
+        ixx="6.5049636783815E-06"
+        ixy="-1.28022090855895E-11"
+        ixz="-2.83914080677337E-10"
+        iyy="1.79658931765907E-06"
+        iyz="-1.60846366473882E-10"
+        izz="6.49720687653235E-06" />
+    </inertial>
+    <visual>
+      <origin
+        xyz="0 0 0"
+        rpy="0 0 0" />
+      <geometry>
+        <mesh
+          filename="file:///home/mo/ws/src/andino/andino_description/meshes/front_left_motor_Link.STL" />
+      </geometry>
+      <material
+        name="">
+        <color
+          rgba="0.298039215686275 0.298039215686275 0.298039215686275 1" />
+      </material>
+    </visual>
+    <collision>
+      <origin
+        xyz="0 0 0"
+        rpy="0 0 0" />
+      <geometry>
+        <mesh
+          filename="file:///home/mo/ws/src/andino/andino_description/meshes/front_left_motor_Link.STL" />
+      </geometry>
+    </collision>
+  </link>
+  <joint
+    name="front_left_motor_joint"
+    type="fixed">
+    <origin
+      xyz="0.14695 0.18351 -0.0138"
+      rpy="0 0 0" />
+    <parent
+      link="base_link" />
+    <child
+      link="front_left_motor_Link" />
+    <axis
+      xyz="0 0 0" />
+  </joint>
+  <link
+    name="front_right_motor_Link">
+    <inertial>
+      <origin
+        xyz="-3.90875860567519E-08 0.0282987057433313 1.94971594275756E-07"
+        rpy="0 0 0" />
+      <mass
+        value="0.0243780634374845" />
+      <inertia
+        ixx="6.50450117035748E-06"
+        ixy="-4.64547734604659E-11"
+        ixz="1.85856843533978E-09"
+        iyy="1.79658931765907E-06"
+        iyz="1.54523151022933E-10"
+        izz="6.49766938455636E-06" />
+    </inertial>
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