Commit message: Update (App) packages and the android app.

File: src/andino/andino_description/urdf/andino.urdf.xacro (robot description, xacro)
@@ -59,5 +59,5 @@
       <geometry>
         <mesh
-          filename="file:///home/mo/ws/src/andino/andino_description/meshes/base_link.STL" />
+          filename="file:///home/jack/ws/src/andino/andino_description/meshes/base_link.STL" />
       </geometry>
       <material
@@ -73,5 +73,5 @@
       <geometry>
         <mesh
-          filename="file:///home/mo/ws/src/andino/andino_description/meshes/base_link.STL" />
+          filename="file:///home/jack/ws/src/andino/andino_description/meshes/base_link.STL" />
       </geometry>
     </collision>
@@ -99,19 +99,19 @@
       <geometry>
         <mesh
-          filename="file:///home/mo/ws/src/andino/andino_description/meshes/left_wheel.STL" />
-      </geometry>
-      <material
-        name="">
-        <color
-          rgba="0.298039215686275 0.298039215686275 0.298039215686275 1" />
-      </material>
-    </visual>
-    <collision>
-      <origin
-        xyz="0 0 0"
-        rpy="0 0 0" />
-      <geometry>
-        <mesh
-          filename="file:///home/mo/ws/src/andino/andino_description/meshes/left_wheel.STL" />
+          filename="file:///home/jack/ws/src/andino/andino_description/meshes/left_wheel.STL" />
+      </geometry>
+      <material
+        name="">
+        <color
+          rgba="0.298039215686275 0.298039215686275 0.298039215686275 1" />
+      </material>
+    </visual>
+    <collision>
+      <origin
+        xyz="0 0 0"
+        rpy="0 0 0" />
+      <geometry>
+        <mesh
+          filename="file:///home/jack/ws/src/andino/andino_description/meshes/left_wheel.STL" />
       </geometry>
     </collision>
@@ -152,19 +152,19 @@
       <geometry>
         <mesh
-          filename="file:///home/mo/ws/src/andino/andino_description/meshes/right_wheel.STL" />
-      </geometry>
-      <material
-        name="">
-        <color
-          rgba="0.298039215686275 0.298039215686275 0.298039215686275 1" />
-      </material>
-    </visual>
-    <collision>
-      <origin
-        xyz="0 0 0"
-        rpy="0 0 0" />
-      <geometry>
-        <mesh
-          filename="file:///home/mo/ws/src/andino/andino_description/meshes/right_wheel.STL" />
+          filename="file:///home/jack/ws/src/andino/andino_description/meshes/right_wheel.STL" />
+      </geometry>
+      <material
+        name="">
+        <color
+          rgba="0.298039215686275 0.298039215686275 0.298039215686275 1" />
+      </material>
+    </visual>
+    <collision>
+      <origin
+        xyz="0 0 0"
+        rpy="0 0 0" />
+      <geometry>
+        <mesh
+          filename="file:///home/jack/ws/src/andino/andino_description/meshes/right_wheel.STL" />
       </geometry>
     </collision>
@@ -205,19 +205,19 @@
       <geometry>
         <mesh
-          filename="file:///home/mo/ws/src/andino/andino_description/meshes/left_back_wheel.STL" />
-      </geometry>
-      <material
-        name="">
-        <color
-          rgba="0.298039215686275 0.298039215686275 0.298039215686275 1" />
-      </material>
-    </visual>
-    <collision>
-      <origin
-        xyz="0 0 0"
-        rpy="0 0 0" />
-      <geometry>
-        <mesh
-          filename="file:///home/mo/ws/src/andino/andino_description/meshes/left_back_wheel.STL" />
+          filename="file:///home/jack/ws/src/andino/andino_description/meshes/left_back_wheel.STL" />
+      </geometry>
+      <material
+        name="">
+        <color
+          rgba="0.298039215686275 0.298039215686275 0.298039215686275 1" />
+      </material>
+    </visual>
+    <collision>
+      <origin
+        xyz="0 0 0"
+        rpy="0 0 0" />
+      <geometry>
+        <mesh
+          filename="file:///home/jack/ws/src/andino/andino_description/meshes/left_back_wheel.STL" />
       </geometry>
     </collision>
@@ -259,19 +259,19 @@
       <geometry>
         <mesh
-          filename="file:///home/mo/ws/src/andino/andino_description/meshes/right_back_wheel.STL" />
-      </geometry>
-      <material
-        name="">
-        <color
-          rgba="0.298039215686275 0.298039215686275 0.298039215686275 1" />
-      </material>
-    </visual>
-    <collision>
-      <origin
-        xyz="0 0 0"
-        rpy="0 0 0" />
-      <geometry>
-        <mesh
-          filename="file:///home/mo/ws/src/andino/andino_description/meshes/right_back_wheel.STL" />
+          filename="file:///home/jack/ws/src/andino/andino_description/meshes/right_back_wheel.STL" />
+      </geometry>
+      <material
+        name="">
+        <color
+          rgba="0.298039215686275 0.298039215686275 0.298039215686275 1" />
+      </material>
+    </visual>
+    <collision>
+      <origin
+        xyz="0 0 0"
+        rpy="0 0 0" />
+      <geometry>
+        <mesh
+          filename="file:///home/jack/ws/src/andino/andino_description/meshes/right_back_wheel.STL" />
       </geometry>
     </collision>
@@ -313,19 +313,19 @@
       <geometry>
         <mesh
-          filename="file:///home/mo/ws/src/andino/andino_description/meshes/front_left_motor_Link.STL" />
-      </geometry>
-      <material
-        name="">
-        <color
-          rgba="0.298039215686275 0.298039215686275 0.298039215686275 1" />
-      </material>
-    </visual>
-    <collision>
-      <origin
-        xyz="0 0 0"
-        rpy="0 0 0" />
-      <geometry>
-        <mesh
-          filename="file:///home/mo/ws/src/andino/andino_description/meshes/front_left_motor_Link.STL" />
+          filename="file:///home/jack/ws/src/andino/andino_description/meshes/front_left_motor_Link.STL" />
+      </geometry>
+      <material
+        name="">
+        <color
+          rgba="0.298039215686275 0.298039215686275 0.298039215686275 1" />
+      </material>
+    </visual>
+    <collision>
+      <origin
+        xyz="0 0 0"
+        rpy="0 0 0" />
+      <geometry>
+        <mesh
+          filename="file:///home/jack/ws/src/andino/andino_description/meshes/front_left_motor_Link.STL" />
       </geometry>
     </collision>
@@ -366,19 +366,19 @@
       <geometry>
         <mesh
-          filename="file:///home/mo/ws/src/andino/andino_description/meshes/front_right_motor_Link.STL" />
-      </geometry>
-      <material
-        name="">
-        <color
-          rgba="0.298039215686275 0.298039215686275 0.298039215686275 1" />
-      </material>
-    </visual>
-    <collision>
-      <origin
-        xyz="0 0 0"
-        rpy="0 0 0" />
-      <geometry>
-        <mesh
-          filename="file:///home/mo/ws/src/andino/andino_description/meshes/front_right_motor_Link.STL" />
+          filename="file:///home/jack/ws/src/andino/andino_description/meshes/front_right_motor_Link.STL" />
+      </geometry>
+      <material
+        name="">
+        <color
+          rgba="0.298039215686275 0.298039215686275 0.298039215686275 1" />
+      </material>
+    </visual>
+    <collision>
+      <origin
+        xyz="0 0 0"
+        rpy="0 0 0" />
+      <geometry>
+        <mesh
+          filename="file:///home/jack/ws/src/andino/andino_description/meshes/front_right_motor_Link.STL" />
       </geometry>
     </collision>
@@ -419,19 +419,19 @@
       <geometry>
         <mesh
-          filename="file:///home/mo/ws/src/andino/andino_description/meshes/rear_left_motor_Link.STL" />
-      </geometry>
-      <material
-        name="">
-        <color
-          rgba="0.298039215686275 0.298039215686275 0.298039215686275 1" />
-      </material>
-    </visual>
-    <collision>
-      <origin
-        xyz="0 0 0"
-        rpy="0 0 0" />
-      <geometry>
-        <mesh
-          filename="file:///home/mo/ws/src/andino/andino_description/meshes/rear_left_motor_Link.STL" />
+          filename="file:///home/jack/ws/src/andino/andino_description/meshes/rear_left_motor_Link.STL" />
+      </geometry>
+      <material
+        name="">
+        <color
+          rgba="0.298039215686275 0.298039215686275 0.298039215686275 1" />
+      </material>
+    </visual>
+    <collision>
+      <origin
+        xyz="0 0 0"
+        rpy="0 0 0" />
+      <geometry>
+        <mesh
+          filename="file:///home/jack/ws/src/andino/andino_description/meshes/rear_left_motor_Link.STL" />
       </geometry>
     </collision>
@@ -472,19 +472,19 @@
       <geometry>
         <mesh
-          filename="file:///home/mo/ws/src/andino/andino_description/meshes/rear_right_motor_joint_Link.STL" />
-      </geometry>
-      <material
-        name="">
-        <color
-          rgba="0.298039215686275 0.298039215686275 0.298039215686275 1" />
-      </material>
-    </visual>
-    <collision>
-      <origin
-        xyz="0 0 0"
-        rpy="0 0 0" />
-      <geometry>
-        <mesh
-          filename="file:///home/mo/ws/src/andino/andino_description/meshes/rear_right_motor_joint_Link.STL" />
+          filename="file:///home/jack/ws/src/andino/andino_description/meshes/rear_right_motor_joint_Link.STL" />
+      </geometry>
+      <material
+        name="">
+        <color
+          rgba="0.298039215686275 0.298039215686275 0.298039215686275 1" />
+      </material>
+    </visual>
+    <collision>
+      <origin
+        xyz="0 0 0"
+        rpy="0 0 0" />
+      <geometry>
+        <mesh
+          filename="file:///home/jack/ws/src/andino/andino_description/meshes/rear_right_motor_joint_Link.STL" />
       </geometry>
     </collision>
@@ -528,5 +528,5 @@
       <geometry>
         <mesh
-          filename="file:///home/mo/ws/src/andino/andino_description/meshes/camera_Link.STL" />
+          filename="file:///home/jack/ws/src/andino/andino_description/meshes/camera_Link.STL" />
       </geometry>
       <material
@@ -542,5 +542,5 @@
       <geometry>
         <mesh
-          filename="file:///home/mo/ws/src/andino/andino_description/meshes/camera_Link.STL" />
+          filename="file:///home/jack/ws/src/andino/andino_description/meshes/camera_Link.STL" />
       </geometry>
     </collision>
@@ -581,5 +581,5 @@
       <geometry>
         <mesh
-          filename="file:///home/mo/ws/src/andino/andino_description/meshes/imu_Link.STL" />
+          filename="file:///home/jack/ws/src/andino/andino_description/meshes/imu_Link.STL" />
       </geometry>
       <material
@@ -595,5 +595,5 @@
       <geometry>
         <mesh
-          filename="file:///home/mo/ws/src/andino/andino_description/meshes/imu_Link.STL" />
+          filename="file:///home/jack/ws/src/andino/andino_description/meshes/imu_Link.STL" />
       </geometry>
     </collision>

Commit message: fix path

File: src/andino/andino_description/urdf/andino.urdf.xacro (robot description, xacro)
@@ -59,5 +59,5 @@
       <geometry>
         <mesh
-          filename="file:///home/jack/ws/src/andino/andino_description/meshes/base_link.STL" />
+          filename="package://andino_description/meshes/base_link.STL" />
       </geometry>
       <material
@@ -73,5 +73,5 @@
       <geometry>
         <mesh
-          filename="file:///home/jack/ws/src/andino/andino_description/meshes/base_link.STL" />
+          filename="package://andino_description/meshes/base_link.STL" />
       </geometry>
     </collision>
@@ -99,19 +99,19 @@
       <geometry>
         <mesh
-          filename="file:///home/jack/ws/src/andino/andino_description/meshes/left_wheel.STL" />
-      </geometry>
-      <material
-        name="">
-        <color
-          rgba="0.298039215686275 0.298039215686275 0.298039215686275 1" />
-      </material>
-    </visual>
-    <collision>
-      <origin
-        xyz="0 0 0"
-        rpy="0 0 0" />
-      <geometry>
-        <mesh
-          filename="file:///home/jack/ws/src/andino/andino_description/meshes/left_wheel.STL" />
+          filename="package://andino_description/meshes/left_wheel.STL" />
+      </geometry>
+      <material
+        name="">
+        <color
+          rgba="0.298039215686275 0.298039215686275 0.298039215686275 1" />
+      </material>
+    </visual>
+    <collision>
+      <origin
+        xyz="0 0 0"
+        rpy="0 0 0" />
+      <geometry>
+        <mesh
+          filename="package://andino_description/meshes/left_wheel.STL" />
       </geometry>
     </collision>
@@ -152,19 +152,19 @@
       <geometry>
         <mesh
-          filename="file:///home/jack/ws/src/andino/andino_description/meshes/right_wheel.STL" />
-      </geometry>
-      <material
-        name="">
-        <color
-          rgba="0.298039215686275 0.298039215686275 0.298039215686275 1" />
-      </material>
-    </visual>
-    <collision>
-      <origin
-        xyz="0 0 0"
-        rpy="0 0 0" />
-      <geometry>
-        <mesh
-          filename="file:///home/jack/ws/src/andino/andino_description/meshes/right_wheel.STL" />
+          filename="package://andino_description/meshes/right_wheel.STL" />
+      </geometry>
+      <material
+        name="">
+        <color
+          rgba="0.298039215686275 0.298039215686275 0.298039215686275 1" />
+      </material>
+    </visual>
+    <collision>
+      <origin
+        xyz="0 0 0"
+        rpy="0 0 0" />
+      <geometry>
+        <mesh
+          filename="package://andino_description/meshes/right_wheel.STL" />
       </geometry>
     </collision>
@@ -205,19 +205,19 @@
       <geometry>
         <mesh
-          filename="file:///home/jack/ws/src/andino/andino_description/meshes/left_back_wheel.STL" />
-      </geometry>
-      <material
-        name="">
-        <color
-          rgba="0.298039215686275 0.298039215686275 0.298039215686275 1" />
-      </material>
-    </visual>
-    <collision>
-      <origin
-        xyz="0 0 0"
-        rpy="0 0 0" />
-      <geometry>
-        <mesh
-          filename="file:///home/jack/ws/src/andino/andino_description/meshes/left_back_wheel.STL" />
+          filename="package://andino_description/meshes/left_back_wheel.STL" />
+      </geometry>
+      <material
+        name="">
+        <color
+          rgba="0.298039215686275 0.298039215686275 0.298039215686275 1" />
+      </material>
+    </visual>
+    <collision>
+      <origin
+        xyz="0 0 0"
+        rpy="0 0 0" />
+      <geometry>
+        <mesh
+          filename="package://andino_description/meshes/left_back_wheel.STL" />
       </geometry>
     </collision>
@@ -259,19 +259,19 @@
       <geometry>
         <mesh
-          filename="file:///home/jack/ws/src/andino/andino_description/meshes/right_back_wheel.STL" />
-      </geometry>
-      <material
-        name="">
-        <color
-          rgba="0.298039215686275 0.298039215686275 0.298039215686275 1" />
-      </material>
-    </visual>
-    <collision>
-      <origin
-        xyz="0 0 0"
-        rpy="0 0 0" />
-      <geometry>
-        <mesh
-          filename="file:///home/jack/ws/src/andino/andino_description/meshes/right_back_wheel.STL" />
+          filename="package://andino_description/meshes/right_back_wheel.STL" />
+      </geometry>
+      <material
+        name="">
+        <color
+          rgba="0.298039215686275 0.298039215686275 0.298039215686275 1" />
+      </material>
+    </visual>
+    <collision>
+      <origin
+        xyz="0 0 0"
+        rpy="0 0 0" />
+      <geometry>
+        <mesh
+          filename="package://andino_description/meshes/right_back_wheel.STL" />
       </geometry>
     </collision>
@@ -313,19 +313,19 @@
       <geometry>
         <mesh
-          filename="file:///home/jack/ws/src/andino/andino_description/meshes/front_left_motor_Link.STL" />
-      </geometry>
-      <material
-        name="">
-        <color
-          rgba="0.298039215686275 0.298039215686275 0.298039215686275 1" />
-      </material>
-    </visual>
-    <collision>
-      <origin
-        xyz="0 0 0"
-        rpy="0 0 0" />
-      <geometry>
-        <mesh
-          filename="file:///home/jack/ws/src/andino/andino_description/meshes/front_left_motor_Link.STL" />
+          filename="package://andino_description/meshes/front_left_motor_Link.STL" />
+      </geometry>
+      <material
+        name="">
+        <color
+          rgba="0.298039215686275 0.298039215686275 0.298039215686275 1" />
+      </material>
+    </visual>
+    <collision>
+      <origin
+        xyz="0 0 0"
+        rpy="0 0 0" />
+      <geometry>
+        <mesh
+          filename="package://andino_description/meshes/front_left_motor_Link.STL" />
       </geometry>
     </collision>
@@ -366,19 +366,19 @@
       <geometry>
         <mesh
-          filename="file:///home/jack/ws/src/andino/andino_description/meshes/front_right_motor_Link.STL" />
-      </geometry>
-      <material
-        name="">
-        <color
-          rgba="0.298039215686275 0.298039215686275 0.298039215686275 1" />
-      </material>
-    </visual>
-    <collision>
-      <origin
-        xyz="0 0 0"
-        rpy="0 0 0" />
-      <geometry>
-        <mesh
-          filename="file:///home/jack/ws/src/andino/andino_description/meshes/front_right_motor_Link.STL" />
+          filename="package://andino_description/meshes/front_right_motor_Link.STL" />
+      </geometry>
+      <material
+        name="">
+        <color
+          rgba="0.298039215686275 0.298039215686275 0.298039215686275 1" />
+      </material>
+    </visual>
+    <collision>
+      <origin
+        xyz="0 0 0"
+        rpy="0 0 0" />
+      <geometry>
+        <mesh
+          filename="package://andino_description/meshes/front_right_motor_Link.STL" />
       </geometry>
     </collision>
@@ -419,19 +419,19 @@
       <geometry>
         <mesh
-          filename="file:///home/jack/ws/src/andino/andino_description/meshes/rear_left_motor_Link.STL" />
-      </geometry>
-      <material
-        name="">
-        <color
-          rgba="0.298039215686275 0.298039215686275 0.298039215686275 1" />
-      </material>
-    </visual>
-    <collision>
-      <origin
-        xyz="0 0 0"
-        rpy="0 0 0" />
-      <geometry>
-        <mesh
-          filename="file:///home/jack/ws/src/andino/andino_description/meshes/rear_left_motor_Link.STL" />
+          filename="package://andino_description/meshes/rear_left_motor_Link.STL" />
+      </geometry>
+      <material
+        name="">
+        <color
+          rgba="0.298039215686275 0.298039215686275 0.298039215686275 1" />
+      </material>
+    </visual>
+    <collision>
+      <origin
+        xyz="0 0 0"
+        rpy="0 0 0" />
+      <geometry>
+        <mesh
+          filename="package://andino_description/meshes/rear_left_motor_Link.STL" />
       </geometry>
     </collision>
@@ -472,19 +472,19 @@
       <geometry>
         <mesh
-          filename="file:///home/jack/ws/src/andino/andino_description/meshes/rear_right_motor_joint_Link.STL" />
-      </geometry>
-      <material
-        name="">
-        <color
-          rgba="0.298039215686275 0.298039215686275 0.298039215686275 1" />
-      </material>
-    </visual>
-    <collision>
-      <origin
-        xyz="0 0 0"
-        rpy="0 0 0" />
-      <geometry>
-        <mesh
-          filename="file:///home/jack/ws/src/andino/andino_description/meshes/rear_right_motor_joint_Link.STL" />
+          filename="package://andino_description/meshes/rear_right_motor_joint_Link.STL" />
+      </geometry>
+      <material
+        name="">
+        <color
+          rgba="0.298039215686275 0.298039215686275 0.298039215686275 1" />
+      </material>
+    </visual>
+    <collision>
+      <origin
+        xyz="0 0 0"
+        rpy="0 0 0" />
+      <geometry>
+        <mesh
+          filename="package://andino_description/meshes/rear_right_motor_joint_Link.STL" />
       </geometry>
     </collision>
@@ -528,5 +528,5 @@
       <geometry>
         <mesh
-          filename="file:///home/jack/ws/src/andino/andino_description/meshes/camera_Link.STL" />
+          filename="package://andino_description/meshes/camera_Link.STL" />
       </geometry>
       <material
@@ -542,5 +542,5 @@
       <geometry>
         <mesh
-          filename="file:///home/jack/ws/src/andino/andino_description/meshes/camera_Link.STL" />
+          filename="package://andino_description/meshes/camera_Link.STL" />
       </geometry>
     </collision>
@@ -581,5 +581,5 @@
       <geometry>
         <mesh
-          filename="file:///home/jack/ws/src/andino/andino_description/meshes/imu_Link.STL" />
+          filename="package://andino_description/meshes/imu_Link.STL" />
       </geometry>
       <material
@@ -595,5 +595,5 @@
       <geometry>
         <mesh
-          filename="file:///home/jack/ws/src/andino/andino_description/meshes/imu_Link.STL" />
+          filename="package://andino_description/meshes/imu_Link.STL" />
       </geometry>
     </collision>
