Commit message: Fix URDF dynamic paths and resolve issues in andino_gz

File: src/andino/andino_description/urdf/andino.urdf.xacro (robot description, xacro)
@@ -2,4 +2,7 @@
 <robot
   name="Delivery Robot_urdf" xmlns:xacro="http://www.ros.org/wiki/xacro">
+  <!-- ========================================================= -->
+  <!-- Properties and Includes -->
+  <!-- ========================================================= -->
   <xacro:property name="package_name" value="andino_description"/>
   <xacro:property name="robot_name" value="andino"/>
@@ -11,7 +14,7 @@
   <xacro:property name="caster_wheel_props" value="${xacro.load_yaml(caster_wheel_yaml)}"/>
   <xacro:arg name="use_fixed_caster" default="True"/>
-  <xacro:arg name="use_real_ros_control" default="True"/>
   <xacro:property name="wheel_yaml" value="$(arg yaml_config_dir)/wheel.yaml" />
   <xacro:property name="wheel_props" value="${xacro.load_yaml(wheel_yaml)}"/>
+  <xacro:property name="wheel_width" value="${wheel_props.get('width', 0.04)}"/>
   <xacro:property name="motor_yaml" value="$(arg yaml_config_dir)/motor.yaml" />
   <xacro:property name="motor_props" value="${xacro.load_yaml(motor_yaml)}"/>
@@ -24,4 +27,18 @@
   <xacro:property name="hardware_yaml" value="$(arg yaml_config_dir)/hardware.yaml" />
   <xacro:property name="hardware_props" value="${xacro.load_yaml(hardware_yaml)}"/>
+  <!-- ========================================================= -->
+  <!-- Macros -->
+  <!-- ========================================================= -->
+  <!-- Macro for wheel inertia to ensure stability -->
+  <xacro:macro name="wheel_inertial" params="mass">
+    <inertial>
+      <origin xyz="0 0 0" rpy="0 0 0"/>
+      <mass value="${mass}"/>
+      <inertia
+        ixx="${mass*(3*wheel_props['radius']*wheel_props['radius']+wheel_width*wheel_width)/12}" ixy="0" ixz="0"
+        iyy="${mass*wheel_props['radius']*wheel_props['radius']/2}" iyz="0"
+        izz="${mass*(3*wheel_props['radius']*wheel_props['radius']+wheel_width*wheel_width)/12}"/>
+    </inertial>
+  </xacro:macro>
   <xacro:macro name="footprint"
                params="wheel_props">
@@ -36,20 +53,18 @@
     </joint>
   </xacro:macro>
+  <!-- ========================================================= -->
+  <!-- Base Link & Footprint -->
+  <!-- ========================================================= -->
     <xacro:footprint wheel_props="${wheel_props}" />
   <link
     name="base_link">
     <inertial>
-      <origin
-        xyz="0.0197110608215278 -0.0027804176800969 0.0969148643167121"
-        rpy="0 0 0" />
-      <mass
-        value="1.71386249919413" />
-      <inertia
-        ixx="0.0231569461000395"
-        ixy="2.50777808928108E-05"
-        ixz="0.000439253426777476"
-        iyy="0.038907074274843"
-        iyz="9.52977406661948E-06"
-        izz="0.0503099220851436" />
+      <!-- Simplified and centered inertia for stability -->
+      <origin xyz="0 0 -0.01" rpy="0 0 0" />
+      <mass value="1.71" />
+      <inertia
+        ixx="0.06" ixy="0" ixz="0"
+        iyy="0.08" iyz="0"
+        izz="0.06" />
     </inertial>
     <visual>
@@ -77,20 +92,10 @@
     </collision>
   </link>
+  <!-- ========================================================= -->
+  <!-- Wheels -->
+  <!-- ========================================================= -->
   <link
     name="left_wheel">
-    <inertial>
-      <origin
-        xyz="-1.43304923483356E-10 0.00578827480780619 2.09625126285085E-10"
-        rpy="0 0 0" />
-      <mass
-        value="0.468152044139992" />
-      <inertia
-        ixx="0.000602353929382081"
-        ixy="-7.18444193596074E-12"
-        ixz="-1.00167587643128E-11"
-        iyy="0.000954241002904411"
-        iyz="1.15813680205067E-12"
-        izz="0.000602353904161843" />
-    </inertial>
+    <xacro:wheel_inertial mass="0.47" />
     <visual>
       <origin
@@ -112,6 +117,5 @@
         rpy="0 0 0" />
       <geometry>
-        <mesh
-          filename="package://andino_description/meshes/left_wheel.STL" />
+        <sphere radius="${wheel_props['radius']}"/>
       </geometry>
     </collision>
@@ -129,21 +133,9 @@
     <axis
       xyz="0 1 0" />
+    <limit effort="500" velocity="100"/>
   </joint>
   <link
     name="right_wheel">
-    <inertial>
-      <origin
-        xyz="-1.16706644348596E-11 -0.00578827480780653 -2.53660450283411E-10"
-        rpy="0 0 0" />
-      <mass
-        value="0.468152044139995" />
-      <inertia
-        ixx="0.000602353913448942"
-        ixy="5.50210245429957E-12"
-        ixz="1.57577941586563E-11"
-        iyy="0.000954241002904415"
-        iyz="4.76280775920882E-12"
-        izz="0.000602353920094988" />
-    </inertial>
+    <xacro:wheel_inertial mass="0.47" />
     <visual>
       <origin
@@ -165,6 +157,5 @@
         rpy="0 0 0" />
       <geometry>
-        <mesh
-          filename="package://andino_description/meshes/right_wheel.STL" />
+        <sphere radius="${wheel_props['radius']}"/>
       </geometry>
     </collision>
@@ -182,21 +173,9 @@
     <axis
       xyz="0 1 0" />
+    <limit effort="500" velocity="100"/>
   </joint>
   <link
     name="left_back_wheel">
-    <inertial>
-      <origin
-        xyz="5.29933874560129E-11 0.00578827480780614 -2.48335936883781E-10"
-        rpy="0 0 0" />
-      <mass
-        value="0.468152044139996" />
-      <inertia
-        ixx="0.00060235391871097"
-        ixy="6.20688903130094E-12"
-        ixz="-1.59872080469483E-11"
-        iyy="0.000954241002904416"
-        iyz="-3.79895060057837E-12"
-        izz="0.000602353914832962" />
-    </inertial>
+    <xacro:wheel_inertial mass="0.47" />
     <visual>
       <origin
@@ -218,6 +197,5 @@
         rpy="0 0 0" />
       <geometry>
-        <mesh
-          filename="package://andino_description/meshes/left_back_wheel.STL" />
+        <sphere radius="${wheel_props['radius']}"/>
       </geometry>
     </collision>
@@ -235,22 +213,10 @@
     <axis
       xyz="0 1 0" />
-            <mimic joint="left_wheel_joint" multiplier="1"/>
+    <limit effort="500" velocity="100"/>
+    <mimic joint="left_wheel_joint" multiplier="1" offset="0"/>
   </joint>
   <link
     name="right_back_wheel">
-    <inertial>
-      <origin
-        xyz="1.05106146008893E-10 -0.00578827480780619 -2.3115340544444E-10"
-        rpy="0 0 0" />
-      <mass
-        value="0.468152044139994" />
-      <inertia
-        ixx="0.000602353902050807"
-        ixy="2.73004690151346E-12"
-        ixz="6.52978696203657E-12"
-        iyy="0.000954241002904414"
-        iyz="6.74568812925498E-12"
-        izz="0.000602353931493122" />
-    </inertial>
+    <xacro:wheel_inertial mass="0.47" />
     <visual>
       <origin
@@ -272,6 +238,5 @@
         rpy="0 0 0" />
       <geometry>
-        <mesh
-          filename="package://andino_description/meshes/right_back_wheel.STL" />
+        <sphere radius="${wheel_props['radius']}"/>
       </geometry>
     </collision>
@@ -288,7 +253,11 @@
       link="right_back_wheel" />
     <axis
-      xyz="0 -1 0" />
-            <mimic joint="right_wheel_joint" multiplier="1"/>
-  </joint>
+      xyz="0 1 0" />
+    <limit effort="500" velocity="100"/>
+    <mimic joint="right_wheel_joint" multiplier="1" offset="0"/>
+  </joint>
+  <!-- ========================================================= -->
+  <!-- Motors -->
+  <!-- ========================================================= -->
   <link
     name="front_left_motor_Link">
@@ -321,13 +290,4 @@
       </material>
     </visual>
-    <collision>
-      <origin
-        xyz="0 0 0"
-        rpy="0 0 0" />
-      <geometry>
-        <mesh
-          filename="package://andino_description/meshes/front_left_motor_Link.STL" />
-      </geometry>
-    </collision>
   </link>
   <joint
@@ -374,13 +334,4 @@
       </material>
     </visual>
-    <collision>
-      <origin
-        xyz="0 0 0"
-        rpy="0 0 0" />
-      <geometry>
-        <mesh
-          filename="package://andino_description/meshes/front_right_motor_Link.STL" />
-      </geometry>
-    </collision>
   </link>
   <joint
@@ -427,13 +378,4 @@
       </material>
     </visual>
-    <collision>
-      <origin
-        xyz="0 0 0"
-        rpy="0 0 0" />
-      <geometry>
-        <mesh
-          filename="package://andino_description/meshes/rear_left_motor_Link.STL" />
-      </geometry>
-    </collision>
   </link>
   <joint
@@ -480,13 +422,4 @@
       </material>
     </visual>
-    <collision>
-      <origin
-        xyz="0 0 0"
-        rpy="0 0 0" />
-      <geometry>
-        <mesh
-          filename="package://andino_description/meshes/rear_right_motor_joint_Link.STL" />
-      </geometry>
-    </collision>
   </link>
   <joint
@@ -503,4 +436,7 @@
       xyz="0 0 0" />
   </joint>
+  <!-- ========================================================= -->
+  <!-- Sensors -->
+  <!-- ========================================================= -->
   <xacro:laser prefix="rplidar" parent_link="base_link"
                    sensor_prop="${sensor_prop}">
@@ -536,13 +472,4 @@
       </material>
     </visual>
-    <collision>
-      <origin
-        xyz="0 0 0"
-        rpy="0 0 0" />
-      <geometry>
-        <mesh
-          filename="package://andino_description/meshes/camera_Link.STL" />
-      </geometry>
-    </collision>
   </link>
   <joint
@@ -589,13 +516,4 @@
       </material>
     </visual>
-    <collision>
-      <origin
-        xyz="0 0 0"
-        rpy="0 0 0" />
-      <geometry>
-        <mesh
-          filename="package://andino_description/meshes/imu_Link.STL" />
-      </geometry>
-    </collision>
   </link>
   <joint
@@ -612,8 +530,8 @@
       xyz="0 0 0" />
   </joint>
-    <!-- ====== ROS 2 Control (hardware interfaces) ====== -->
-  <xacro:if value="$(arg use_real_ros_control)">
-    <xacro:include filename="$(find ${package_name})/urdf/include/andino_control.urdf.xacro" />
-    <xacro:control hardware_props="${hardware_props}" />
-  </xacro:if>
+  <!-- ========================================================= -->
+  <!-- ROS 2 Control (hardware interfaces) -->
+  <!-- ========================================================= -->
+  <xacro:include filename="$(find ${package_name})/urdf/include/andino_control.urdf.xacro" />
+  <xacro:control hardware_props="${hardware_props}" />
 </robot>

File: src/andino_gz/andino_gz/urdf/andino_gz.urdf.xacro (robot description, xacro)
@@ -2,4 +2,68 @@
 <robot xmlns:xacro="http://www.ros.org/wiki/xacro" name="andino">
   <xacro:include filename="$(find andino_description)/urdf/andino.urdf.xacro"/>
+  <gazebo>
+    <!-- ========================================================= -->
+    <!-- Gazebo Properties (Moved from andino.urdf.xacro) -->
+    <!-- ========================================================= -->
+  </gazebo>
+  <gazebo reference="left_wheel">
+    <mu1>1.0</mu1>
+    <mu2>1.0</mu2>
+    <fdir1>1 0 0</fdir1>
+    <kp>1000000.0</kp>
+    <kd>10.0</kd>
+    <minDepth>0.001</minDepth>
+  </gazebo>
+  <gazebo reference="right_wheel">
+    <mu1>1.0</mu1>
+    <mu2>1.0</mu2>
+    <fdir1>1 0 0</fdir1>
+    <kp>1000000.0</kp>
+    <kd>10.0</kd>
+    <minDepth>0.001</minDepth>
+  </gazebo>
+  <gazebo reference="left_back_wheel">
+    <mu1>0.0</mu1>
+    <mu2>0.0</mu2>
+    <fdir1>1 0 0</fdir1>
+    <kp>1000000.0</kp>
+    <kd>10.0</kd>
+    <minDepth>0.001</minDepth>
+  </gazebo>
+  <gazebo reference="right_back_wheel">
+    <mu1>0.0</mu1>
+    <mu2>0.0</mu2>
+    <fdir1>1 0 0</fdir1>
+    <kp>1000000.0</kp>
+    <kd>10.0</kd>
+    <minDepth>0.001</minDepth>
+  </gazebo>
+  <!-- Gazebo Camera Plugin (Classic) -->
+  <gazebo reference="camera_Link">
+    <sensor type="camera" name="camera_classic">
+      <update_rate>30.0</update_rate>
+      <camera name="head">
+        <horizontal_fov>1.3962634</horizontal_fov>
+        <image>
+          <width>640</width>
+          <height>480</height>
+          <format>R8G8B8</format>
+        </image>
+        <clip>
+          <near>0.02</near>
+          <far>300</far>
+        </clip>
+      </camera>
+      <plugin name="camera_controller" filename="libgazebo_ros_camera.so">
+        <alwaysOn>true</alwaysOn>
+        <updateRate>0.0</updateRate>
+        <cameraName>camera</cameraName>
+        <imageTopicName>/image_raw</imageTopicName>
+        <cameraInfoTopicName>/camera_info</cameraInfoTopicName>
+        <frameName>camera_Link</frameName>
+        <hackBaseline>0.07</hackBaseline>
+      </plugin>
+    </sensor>
+  </gazebo>
   <gazebo>
     <plugin
@@ -38,6 +102,6 @@
       <joint_name>left_wheel_joint</joint_name>
       <joint_name>right_wheel_joint</joint_name>
-      <joint_name>caster_wheel_joint</joint_name>
-      <joint_name>caster_rotation_joint</joint_name>
+      <joint_name>left_back_wheel_joint</joint_name>
+      <joint_name>right_back_wheel_joint</joint_name>
     </plugin>
   </gazebo>
@@ -73,7 +137,7 @@
     </plugin>
   </gazebo>
-  <gazebo reference="camera_link">
+  <gazebo reference="camera_Link">
     <sensor name="camera" type="camera">
-      <gz_frame_id>camera_link</gz_frame_id>
+      <gz_frame_id>camera_Link</gz_frame_id>
       <camera>
         <horizontal_fov>1.047</horizontal_fov>

File: src/andino_gz/andino_gz/urdf/include/andino_materials.xacro (robot description, xacro)
@@ -5,6 +5,6 @@
       <visual>
         <material>
-          <ambient>0.0 0.0 1.0 1.0</ambient>
-          <diffuse>0.0 0.0 1.0 1.0</diffuse>
+          <ambient>0.5 0.5 0.5 1.0</ambient>
+          <diffuse>0.5 0.5 0.5 1.0</diffuse>
           <specular>0.1 0.1 0.1 1.0</specular>
           <emissive>0.0 0.0 0.0 1.0</emissive>
@@ -26,6 +26,6 @@
       <visual>
         <material>
-          <ambient>0.1 0.1 0.1 1.0</ambient>
-          <diffuse>0.02 0.02 0.02 1.0</diffuse>
+          <ambient>0.0 0.0 0.0 1.0</ambient>
+          <diffuse>0.0 0.0 0.0 1.0</diffuse>
           <specular>0.1 0.1 0.1 1.0</specular>
           <emissive>0.0 0.0 0.0 1.0</emissive>
@@ -36,6 +36,26 @@
       <visual>
         <material>
-          <ambient>0.1 0.1 0.1 1.0</ambient>
-          <diffuse>0.02 0.02 0.02 1.0</diffuse>
+          <ambient>0.0 0.0 0.0 1.0</ambient>
+          <diffuse>0.0 0.0 0.0 1.0</diffuse>
+          <specular>0.1 0.1 0.1 1.0</specular>
+          <emissive>0.0 0.0 0.0 1.0</emissive>
+        </material>
+      </visual>
+    </gazebo>
+    <gazebo reference="left_back_wheel">
+      <visual>
+        <material>
+          <ambient>0.0 0.0 0.0 1.0</ambient>
+          <diffuse>0.0 0.0 0.0 1.0</diffuse>
+          <specular>0.1 0.1 0.1 1.0</specular>
+          <emissive>0.0 0.0 0.0 1.0</emissive>
+        </material>
+      </visual>
+    </gazebo>
+    <gazebo reference="right_back_wheel">
+      <visual>
+        <material>
+          <ambient>0.0 0.0 0.0 1.0</ambient>
+          <diffuse>0.0 0.0 0.0 1.0</diffuse>
           <specular>0.1 0.1 0.1 1.0</specular>
           <emissive>0.0 0.0 0.0 1.0</emissive>
@@ -96,5 +116,5 @@
     </gazebo>
     <!-- Camera -->
-    <gazebo reference="camera_link">
+    <gazebo reference="camera_Link">
       <visual>
         <material>
