Commit message: chore: Clean up firmware dependencies and update robot configuration, app build artifacts, and Python scripts.

File: src/andino_gz/andino_gz/urdf/andino_gz.urdf.xacro (robot description, xacro)
@@ -1,10 +1,541 @@
 <?xml version="1.0"?>
-<robot xmlns:xacro="http://www.ros.org/wiki/xacro" name="andino">
-  <xacro:include filename="$(find andino_description)/urdf/andino.urdf.xacro"/>
-  <gazebo>
-    <!-- ========================================================= -->
-    <!-- Gazebo Properties (Moved from andino.urdf.xacro) -->
-    <!-- ========================================================= -->
-  </gazebo>
+<robot
+  name="Delivery Robot_urdf" xmlns:xacro="http://www.ros.org/wiki/xacro">
+  <!-- ========================================================= -->
+  <!-- Properties and Includes -->
+  <!-- ========================================================= -->
+  <xacro:property name="package_name" value="andino_description"/>
+  <xacro:property name="robot_name" value="andino"/>
+  <xacro:include filename="$(find ${package_name})/urdf/include/common_macros.urdf.xacro" />
+  <xacro:include filename="$(find ${package_name})/urdf/include/common_sensors.urdf.xacro" />
+  <xacro:include filename="$(find ${package_name})/urdf/include/andino_caster_macro.urdf.xacro" />
+  <xacro:arg name="yaml_config_dir" default="$(find ${package_name})/config/${robot_name}" />
+  <xacro:property name="caster_wheel_yaml" value="$(arg yaml_config_dir)/caster_wheel.yaml" />
+  <xacro:property name="caster_wheel_props" value="${xacro.load_yaml(caster_wheel_yaml)}"/>
+  <xacro:arg name="use_fixed_caster" default="True"/>
+  <xacro:property name="wheel_yaml" value="$(arg yaml_config_dir)/wheel.yaml" />
+  <xacro:property name="wheel_props" value="${xacro.load_yaml(wheel_yaml)}"/>
+  <xacro:property name="wheel_width" value="${wheel_props.get('width', 0.04)}"/>
+  <xacro:property name="motor_yaml" value="$(arg yaml_config_dir)/motor.yaml" />
+  <xacro:property name="motor_props" value="${xacro.load_yaml(motor_yaml)}"/>
+  <xacro:property name="base_yaml" value="$(arg yaml_config_dir)/base.yaml" />
+  <xacro:property name="base_props" value="${xacro.load_yaml(base_yaml)}"/>
+  <xacro:property name="second_base_yaml" value="$(arg yaml_config_dir)/second_base.yaml" />
+  <xacro:property name="second_base_props" value="${xacro.load_yaml(second_base_yaml)}"/>
+  <xacro:property name="sensor_yaml" value="$(arg yaml_config_dir)/sensors.yaml" />
+  <xacro:property name="sensor_prop" value="${xacro.load_yaml(sensor_yaml)}"/>
+  <xacro:property name="hardware_yaml" value="$(arg yaml_config_dir)/hardware.yaml" />
+  <xacro:property name="hardware_props" value="${xacro.load_yaml(hardware_yaml)}"/>
+  <!-- ========================================================= -->
+  <!-- Macros -->
+  <!-- ========================================================= -->
+  <!-- Macro for wheel inertia to ensure stability -->
+  <xacro:macro name="wheel_inertial" params="mass">
+    <inertial>
+      <origin xyz="0 0 0" rpy="0 0 0"/>
+      <mass value="${mass}"/>
+      <inertia
+        ixx="${mass*(3*wheel_props['radius']*wheel_props['radius']+wheel_width*wheel_width)/12}" ixy="0" ixz="0"
+        iyy="${mass*wheel_props['radius']*wheel_props['radius']/2}" iyz="0"
+        izz="${mass*(3*wheel_props['radius']*wheel_props['radius']+wheel_width*wheel_width)/12}"/>
+    </inertial>
+  </xacro:macro>
+  <xacro:macro name="footprint"
+               params="wheel_props">
+    <!-- Base-Footprint -->
+    <!-- base_footprint is a fictitious link(frame) that is on the ground right below base_link origin -->
+    <link name="base_footprint" />
+    <!-- Joint to connect base_footprint with base_link -->
+    <joint name="base_footprint_joint" type="fixed">
+      <parent link="base_link"/>
+      <child link="base_footprint" />
+      <origin xyz="0 0 ${-(wheel_props['radius'] - wheel_props['z_offset'])}" rpy="0 0 0" />
+    </joint>
+  </xacro:macro>
+  <!-- ========================================================= -->
+  <!-- Base Link & Footprint -->
+  <!-- ========================================================= -->
+    <xacro:footprint wheel_props="${wheel_props}" />
+  <link
+    name="base_link">
+    <inertial>
+      <!-- Simplified and centered inertia for stability -->
+      <origin xyz="0 0 -0.01" rpy="0 0 0" />
+      <mass value="1.71" />
+      <inertia
+        ixx="0.06" ixy="0" ixz="0"
+        iyy="0.08" iyz="0"
+        izz="0.06" />
+    </inertial>
+    <visual>
+      <origin
+        xyz="0 0 0"
+        rpy="0 0 0" />
+      <geometry>
+        <mesh
+          filename="package://andino_description/meshes/base_link.STL" />
+      </geometry>
+      <material
+        name="">
+        <color
+          rgba="0 0 0 1" />
+      </material>
+    </visual>
+    <collision>
+      <origin
+        xyz="0 0 0"
+        rpy="0 0 0" />
+      <geometry>
+        <mesh
+          filename="package://andino_description/meshes/base_link.STL" />
+      </geometry>
+    </collision>
+  </link>
+  <!-- ========================================================= -->
+  <!-- Wheels -->
+  <!-- ========================================================= -->
+  <link
+    name="left_wheel">
+    <xacro:wheel_inertial mass="0.47" />
+    <visual>
+      <origin
+        xyz="0 0 0"
+        rpy="0 0 0" />
+      <geometry>
+        <mesh
+          filename="package://andino_description/meshes/left_wheel.STL" />
+      </geometry>
+      <material
+        name="">
+        <color
+          rgba="0.298039215686275 0.298039215686275 0.298039215686275 1" />
+      </material>
+    </visual>
+    <collision>
+      <origin
+        xyz="0 0 0"
+        rpy="0 0 0" />
+      <geometry>
+        <sphere radius="${wheel_props['radius']}"/>
+      </geometry>
+    </collision>
+  </link>
+  <joint
+    name="left_wheel_joint"
+    type="continuous">
+    <origin
+      xyz="0.14695 0.20151 -0.0138"
+      rpy="0 0 0" />
+    <parent
+      link="base_link" />
+    <child
+      link="left_wheel" />
+    <axis
+      xyz="0 1 0" />
+    <limit effort="500" velocity="100"/>
+  </joint>
+  <link
+    name="right_wheel">
+    <xacro:wheel_inertial mass="0.47" />
+    <visual>
+      <origin
+        xyz="0 0 0"
+        rpy="0 0 0" />
+      <geometry>
+        <mesh
+          filename="package://andino_description/meshes/right_wheel.STL" />
+      </geometry>
+      <material
+        name="">
+        <color
+          rgba="0.298039215686275 0.298039215686275 0.298039215686275 1" />
+      </material>
+    </visual>
+    <collision>
+      <origin
+        xyz="0 0 0"
+        rpy="0 0 0" />
+      <geometry>
+        <sphere radius="${wheel_props['radius']}"/>
+      </geometry>
+    </collision>
+  </link>
+  <joint
+    name="right_wheel_joint"
+    type="continuous">
+    <origin
+      xyz="0.14695 -0.20149 -0.0138"
+      rpy="0 0 0" />
+    <parent
+      link="base_link" />
+    <child
+      link="right_wheel" />
+    <axis
+      xyz="0 1 0" />
+    <limit effort="500" velocity="100"/>
+  </joint>
+  <link
+    name="left_back_wheel">
+    <xacro:wheel_inertial mass="0.47" />
+    <visual>
+      <origin
+        xyz="0 0 0"
+        rpy="0 0 0" />
+      <geometry>
+        <mesh
+          filename="package://andino_description/meshes/left_back_wheel.STL" />
+      </geometry>
+      <material
+        name="">
+        <color
+          rgba="0.298039215686275 0.298039215686275 0.298039215686275 1" />
+      </material>
+    </visual>
+    <collision>
+      <origin
+        xyz="0 0 0"
+        rpy="0 0 0" />
+      <geometry>
+        <sphere radius="${wheel_props['radius']}"/>
+      </geometry>
+    </collision>
+  </link>
+  <joint
+    name="left_back_wheel_joint"
+    type="continuous">
+    <origin
+      xyz="-0.14305 0.20001 -0.0138"
+      rpy="0 0 0" />
+    <parent
+      link="base_link" />
+    <child
+      link="left_back_wheel" />
+    <axis
+      xyz="0 1 0" />
+    <limit effort="500" velocity="100"/>
+    <mimic joint="left_wheel_joint" multiplier="1" offset="0"/>
+  </joint>
+  <link
+    name="right_back_wheel">
+    <xacro:wheel_inertial mass="0.47" />
+    <visual>
+      <origin
+        xyz="0 0 0"
+        rpy="0 0 0" />
+      <geometry>
+        <mesh
+          filename="package://andino_description/meshes/right_back_wheel.STL" />
+      </geometry>
+      <material
+        name="">
+        <color
+          rgba="0.298039215686275 0.298039215686275 0.298039215686275 1" />
+      </material>
+    </visual>
+    <collision>
+      <origin
+        xyz="0 0 0"
+        rpy="0 0 0" />
+      <geometry>
+        <sphere radius="${wheel_props['radius']}"/>
+      </geometry>
+    </collision>
+  </link>
+  <joint
+    name="right_back_wheel_joint"
+    type="continuous">
+    <origin
+      xyz="-0.14305 -0.20149 -0.0138"
+      rpy="0 0 0" />
+    <parent
+      link="base_link" />
+    <child
+      link="right_back_wheel" />
+    <axis
+      xyz="0 1 0" />
+    <limit effort="500" velocity="100"/>
+    <mimic joint="right_wheel_joint" multiplier="1" offset="0"/>
+  </joint>
+  <!-- ========================================================= -->
+  <!-- Motors -->
+  <!-- ========================================================= -->
+  <link
+    name="front_left_motor_Link">
+    <inertial>
+      <origin
+        xyz="-2.93427859787698E-09 -0.0282987057433313 1.98829454782501E-07"
+        rpy="0 0 0" />
+      <mass
+        value="0.0243780634374845" />
+      <inertia
+        ixx="6.5049636783815E-06"
+        ixy="-1.28022090855895E-11"
+        ixz="-2.83914080677337E-10"
+        iyy="1.79658931765907E-06"
+        iyz="-1.60846366473882E-10"
+        izz="6.49720687653235E-06" />
+    </inertial>
+    <visual>
+      <origin
+        xyz="0 0 0"
+        rpy="0 0 0" />
+      <geometry>
+        <mesh
+          filename="package://andino_description/meshes/front_left_motor_Link.STL" />
+      </geometry>
+      <material
+        name="">
+        <color
+          rgba="0.298039215686275 0.298039215686275 0.298039215686275 1" />
+      </material>
+    </visual>
+  </link>
+  <joint
+    name="front_left_motor_joint"
+    type="fixed">
+    <origin
+      xyz="0.14695 0.18351 -0.0138"
+      rpy="0 0 0" />
+    <parent
+      link="base_link" />
+    <child
+      link="front_left_motor_Link" />
+    <axis
+      xyz="0 0 0" />
+  </joint>
+  <link
+    name="front_right_motor_Link">
+    <inertial>
+      <origin
+        xyz="-3.90875860567519E-08 0.0282987057433313 1.94971594275756E-07"
+        rpy="0 0 0" />
+      <mass
+        value="0.0243780634374845" />
+      <inertia
+        ixx="6.50450117035748E-06"
+        ixy="-4.64547734604659E-11"
+        ixz="1.85856843533978E-09"
+        iyy="1.79658931765907E-06"
+        iyz="1.54523151022933E-10"
+        izz="6.49766938455636E-06" />
+    </inertial>
+    <visual>
+      <origin
+        xyz="0 0 0"
+        rpy="0 0 0" />
+      <geometry>
+        <mesh
+          filename="package://andino_description/meshes/front_right_motor_Link.STL" />
+      </geometry>
+      <material
+        name="">
+        <color
+          rgba="0.298039215686275 0.298039215686275 0.298039215686275 1" />
+      </material>
+    </visual>
+  </link>
+  <joint
+    name="front_right_motor_joint"
+    type="fixed">
+    <origin
+      xyz="0.14695 -0.18349 -0.0138"
+      rpy="0 0 0" />
+    <parent
+      link="base_link" />
+    <child
+      link="front_right_motor_Link" />
+    <axis
+      xyz="0 0 0" />
+  </joint>
+  <link
+    name="rear_left_motor_Link">
+    <inertial>
+      <origin
+        xyz="-2.93427060427121E-09 -0.0257987057433852 1.98829458026434E-07"
+        rpy="0 0 0" />
+      <mass
+        value="0.0243780634374845" />
+      <inertia
+        ixx="6.5049636783815E-06"
+        ixy="-1.28022090855905E-11"
+        ixz="-2.83914080677331E-10"
+        iyy="1.79658931765907E-06"
+        iyz="-1.60846366473941E-10"
+        izz="6.49720687653235E-06" />
+    </inertial>
+    <visual>
+      <origin
+        xyz="0 0 0"
+        rpy="0 0 0" />
+      <geometry>
+        <mesh
+          filename="package://andino_description/meshes/rear_left_motor_Link.STL" />
+      </geometry>
+      <material
+        name="">
+        <color
+          rgba="0.298039215686275 0.298039215686275 0.298039215686275 1" />
+      </material>
+    </visual>
+  </link>
+  <joint
+    name="rear_left_motor_joint"
+    type="fixed">
+    <origin
+      xyz="-0.14305 0.18101 -0.0138"
+      rpy="0 0 0" />
+    <parent
+      link="base_link" />
+    <child
+      link="rear_left_motor_Link" />
+    <axis
+      xyz="0 0 0" />
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
Commit message: add ultrasonic

File: src/andino/andino_description/urdf/andino.urdf.xacro (robot description, xacro)
@@ -627,5 +627,34 @@
       xyz="0 0 0" />
   </joint>
-    <!-- ====== ROS 2 Control (hardware interfaces) ====== -->
+  <!-- ========================================================= -->
+  <!-- Ultrasonic Sensor  -->
+  <!-- ========================================================= -->
+  <link name="ultrasonic_sensor_link">
+    <visual>
+      <origin xyz="0 0 0" rpy="0 0 0"/>
+      <geometry>
+        <box size="0.02 0.04 0.02"/>
+      </geometry>
+      <material name="blue">
+        <color rgba="0.0 0.0 1.0 1.0"/>
+      </material>
+    </visual>
+    <collision>
+      <origin xyz="0 0 0" rpy="0 0 0"/>
+      <geometry>
+        <box size="0.02 0.04 0.02"/>
+      </geometry>
+    </collision>
+    <inertial>
+      <mass value="0.01"/>
+      <inertia ixx="1e-5" ixy="0" ixz="0" iyy="1e-5" iyz="0" izz="1e-5"/>
+    </inertial>
+  </link>
+  <joint name="ultrasonic_joint" type="fixed">
+    <parent link="base_link"/>
+    <child link="ultrasonic_sensor_link"/>
+    <origin xyz="0.22 0 0.02" rpy="0 0 0"/>
+  </joint>
+  <!-- ====== ROS 2 Control (hardware interfaces) ====== -->
   <xacro:if value="$(arg use_real_ros_control)">
     <xacro:include filename="$(find ${package_name})/urdf/include/andino_control.urdf.xacro" />

File: src/andino/andino_description/urdf/include/andino_control.urdf.xacro (robot description, xacro)
@@ -33,4 +33,7 @@
         <state_interface name="position"/>
       </joint>
+      <joint name="ultrasonic_sensor">
+        <state_interface name="range"/>
+      </joint>
     </ros2_control>
   </xacro:macro>

File: src/andino_gz/andino_gz/urdf/andino_gz.urdf.xacro (robot description, xacro)
@@ -529,4 +529,33 @@
     <axis
       xyz="0 0 0" />
+  </joint>
+  <!-- ========================================================= -->
+  <!-- Ultrasonic Sensor  -->
+  <!-- ========================================================= -->
+  <link name="ultrasonic_sensor_link">
+    <visual>
+      <origin xyz="0 0 0" rpy="0 0 0"/>
+      <geometry>
+        <box size="0.02 0.04 0.02"/>
+      </geometry>
+      <material name="blue">
+        <color rgba="0.0 0.0 1.0 1.0"/>
+      </material>
+    </visual>
+    <collision>
+      <origin xyz="0 0 0" rpy="0 0 0"/>
+      <geometry>
+        <box size="0.02 0.04 0.02"/>
+      </geometry>
+    </collision>
+    <inertial>
+      <mass value="0.01"/>
+      <inertia ixx="1e-5" ixy="0" ixz="0" iyy="1e-5" iyz="0" izz="1e-5"/>
+    </inertial>
+  </link>
+  <joint name="ultrasonic_joint" type="fixed">
+    <parent link="base_link"/>
+    <child link="ultrasonic_sensor_link"/>
+    <origin xyz="0.22 0 0.02" rpy="0 0 0"/>
   </joint>
   <!-- ========================================================= -->
@@ -664,4 +693,39 @@
     </sensor>
   </gazebo>
+  <gazebo reference="ultrasonic_sensor_link">
+    <sensor name="ultrasonic_sensor" type="gpu_lidar">
+      <gz_frame_id>ultrasonic_sensor_link</gz_frame_id>
+      <ray>
+        <scan>
+          <horizontal>
+            <samples>5</samples>
+            <resolution>1</resolution>
+            <min_angle>-0.26</min_angle>
+            <max_angle>0.26</max_angle>
+          </horizontal>
+          <vertical>
+            <samples>5</samples>
+            <resolution>1</resolution>
+            <min_angle>-0.26</min_angle>
+            <max_angle>0.26</max_angle>
+          </vertical>
+        </scan>
+        <range>
+          <min>0.02</min>
+          <max>4.0</max>
+          <resolution>0.01</resolution>
+        </range>
+        <noise>
+          <type>gaussian</type>
+          <mean>0.0</mean>
+          <stddev>0.01</stddev>
+        </noise>
+      </ray>
+      <always_on>true</always_on>
+      <visualize>true</visualize>
+      <update_rate>10.0</update_rate>
+      <topic>ultrasonic_sensor/range</topic>
+    </sensor>
+  </gazebo>
   <xacro:include filename="$(find andino_gz)/urdf/include/andino_materials.xacro"/>
 </robot>

Commit message: feat: Update MPU6050 library dependencies, remove NewPing, and refine various robot configuration and firmware files.

File: src/andino/andino_description/urdf/andino.urdf.xacro (robot description, xacro)
@@ -627,34 +627,5 @@
       xyz="0 0 0" />
   </joint>
-  <!-- ========================================================= -->
-  <!-- Ultrasonic Sensor  -->
-  <!-- ========================================================= -->
-  <link name="ultrasonic_sensor_link">
-    <visual>
-      <origin xyz="0 0 0" rpy="0 0 0"/>
-      <geometry>
-        <box size="0.02 0.04 0.02"/>
-      </geometry>
-      <material name="blue">
-        <color rgba="0.0 0.0 1.0 1.0"/>
-      </material>
-    </visual>
-    <collision>
-      <origin xyz="0 0 0" rpy="0 0 0"/>
-      <geometry>
-        <box size="0.02 0.04 0.02"/>
-      </geometry>
-    </collision>
-    <inertial>
-      <mass value="0.01"/>
-      <inertia ixx="1e-5" ixy="0" ixz="0" iyy="1e-5" iyz="0" izz="1e-5"/>
-    </inertial>
-  </link>
-  <joint name="ultrasonic_joint" type="fixed">
-    <parent link="base_link"/>
-    <child link="ultrasonic_sensor_link"/>
-    <origin xyz="0.22 0 0.02" rpy="0 0 0"/>
-  </joint>
-  <!-- ====== ROS 2 Control (hardware interfaces) ====== -->
+    <!-- ====== ROS 2 Control (hardware interfaces) ====== -->
   <xacro:if value="$(arg use_real_ros_control)">
     <xacro:include filename="$(find ${package_name})/urdf/include/andino_control.urdf.xacro" />

File: src/andino/andino_description/urdf/include/andino_control.urdf.xacro (robot description, xacro)
@@ -33,7 +33,4 @@
         <state_interface name="position"/>
       </joint>
-      <joint name="ultrasonic_joint">
-        <state_interface name="range"/>
-      </joint>
     </ros2_control>
   </xacro:macro>
